File: MOS CPU Replacement.kicad_pcb (KiCad board)
At the start: 4 copper layers, 28.2 x 56.4 mm, 70 parts, among them J1 8500/6510T/8501, J4 8502, U1 6502, U10 HCT126, U11 HCT126, U12 HCT126, U13 LVC1G373, U2 HCT245, U3 HCT245, U4 HCT245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

Commit message: Update to Rev2
Parts:
- J1: value 8500/6510T/8501 -> 6510/6510T/8501
- moved REF** 0.74 mm to (164.3, 129.9)
- moved D11 0.53 mm to (145.7, 129.8)
- moved D12 0.53 mm to (148.9, 129.8)
- moved D13 0.53 mm to (152.2, 129.8)
- moved D14 0.53 mm to (155.5, 129.8)
- moved D15 0.53 mm to (158.8, 129.8)
- moved JP22 0.38 mm to (164.5, 127.9), turned to 180 degrees
- moved JP19 0.38 mm to (164.5, 125.3)
- moved JP23 0.38 mm to (164.5, 122.8)
- moved LOGO1 0.25 mm to (165.6, 128.3)
- moved D1 0.18 mm to (141.4, 97.8)
- moved D10 0.18 mm to (141.4, 127.7)
- moved D2 0.18 mm to (141.4, 101.1)
- moved D3 0.18 mm to (141.4, 104.4)
- moved D4 0.18 mm to (141.4, 107.7)
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Connections:
- U1 pad 3: (no net) -> unconnected-(U1-Pad3)
- U1 pad 35: (no net) -> unconnected-(U1-Pad35)
- U1 pad 39: /PHI2 -> Net-(U1-Pad39)
- U1 pad 5: (no net) -> unconnected-(U1-Pad5)
- U1 pad 7: (no net) -> unconnected-(U1-Pad7)
- U10 pad 11: (no net) -> /PHI2
- U10 pad 12: VCC -> Net-(U1-Pad39)
- U9 pad 12: (no net) -> unconnected-(U9-Pad12)
- U9 pad 13: (no net) -> unconnected-(U9-Pad13)
- U9 pad 14: (no net) -> unconnected-(U9-Pad14)
- U9 pad 15: (no net) -> unconnected-(U9-Pad15)
Routing:
- net Net-(U1-Pad39): track 0.00 -> 41.5 mm, vias 0 -> 1
- net /PHI2: track 3.96 -> 31.2 mm, vias 0 -> 1
- net /CA14: track 23.2 -> 28.3 mm, vias 0 -> 2
- net GND: track 196.4 -> 194.4 mm
- net VCC: track 269.2 -> 267.5 mm
- net /CA1: track 19.9 -> 21.0 mm
- net /A11: track 9.13 -> 9.93 mm
- net Net-(J1-Pad24): track 20.7 -> 19.9 mm
- net /CA15: track 23.6 -> 23.0 mm
- net /CA11: track 15.1 -> 14.5 mm
- net /P0: track 26.5 -> 26.0 mm
- net /~{RW}: track 47.2 -> 46.7 mm
Other:
- board size 28.2 x 56.4 mm -> 28.2 x 56 mm
- board text added: "Cut 'W' jumper if using W65C02. Leave connected otherwise."
- board text added: "Rev2"
- board text added: "Solder all jumpers that contain the desired letter."
- board text removed: "Cut 'W' jumper if using W65C02."
- board text removed: "JLCJLCJLCJLC"
- board text removed: "Rev1"
