File: MOS CPU Replacement.kicad_sch (KiCad schematic)
At the start: 67 parts, among them J1 6510/6510T/8501, J4 8502, U1 6502, U10 HCT126, U11 HCT126, U12 HCT126, U13 LVC1G373, U2 HCT245, U3 HCT245, U4 HCT245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

Commit message: Update to Rev2
Parts:
- U13: footprint Package_TO_SOT_SMD:SOT-23-6 -> Package_TO_SOT_SMD:SOT-363_SC-70-6
Connections:
- net PHI2: now also U10.11; no longer U1.39 (PHI2OUT)
- net VCC: no longer U10.12
- new net: U1.39 (PHI2OUT), U10.12
- no-connect marks 9 -> 8
Other:
- note added: "Clock buffer added in Rev2. Should fix C64 compatibility issues, and maybe some others. Thanks to Ray of Retro Tech Insanity."
- moved on the sheet: U10D
